Commit message: abc

File: resources/iiwa/iiwa_spherized.urdf (robot description, URDF)
Before this commit: robot iiwa14, 21 links, 20 joints
Links:
- link base: geometry collision sphere radius=0.07; visual mesh filename=link_0.obj
- link link1: geometry collision sphere radius=0.07; collision sphere radius=0.07
- link link2: geometry collision sphere radius=0.065; collision sphere radius=0.065
- link link3: geometry collision sphere radius=0.055; collision sphere radius=0.055
- link link4: geometry collision sphere radius=0.06; collision sphere radius=0.06
- link link5: geometry collision sphere radius=0.035; collision sphere radius=0.035
- link link6: geometry collision sphere radius=0.055; collision sphere radius=0.065
- link link7: geometry collision sphere radius=0.02; visual mesh filename=link_7.obj
