Commit message: update iiwa spherical model

File: cricket/resources/iiwa/iiwa_spherized.urdf (robot description, URDF)
Before this commit: robot iiwa, 21 links, 20 joints
Links:
- removed link iiwa_link_0
- removed link iiwa_link_1
- removed link iiwa_link_2
- removed link iiwa_link_3
- removed link iiwa_link_4
- removed link iiwa_link_5
- removed link iiwa_link_6
- removed link iiwa_link_7
- removed link world
- added link attachment_site
- added link base, mass 5; collision sphere radius=0.07; visual mesh filename=assets/link_0.obj
- added link link1, mass 5.76; collision sphere radius=0.07; collision sphere radius=0.07
- added link link2, mass 6.35; collision sphere radius=0.065; collision sphere radius=0.065
- added link link3, mass 3.5; collision sphere radius=0.055; collision sphere radius=0.055
- added link link4, mass 3.5; collision sphere radius=0.06; collision sphere radius=0.06
- added link link5, mass 3.5; collision sphere radius=0.035; collision sphere radius=0.035
- added link link6, mass 1.8; collision sphere radius=0.055; collision sphere radius=0.065
- added link link7, mass 1.2; collision sphere radius=0.02; visual mesh filename=assets/link_7.obj
Joints:
- removed joint iiwa_joint_1
- removed joint iiwa_joint_2
- removed joint iiwa_joint_3
- removed joint iiwa_joint_4
- removed joint iiwa_joint_5
- removed joint iiwa_joint_6
- removed joint iiwa_joint_7
- removed joint world_iiwa_joint
- added joint attachment_joint: type fixed, parent link7, child attachment_site, origin xyz=0 0 0.045 rpy=0 0 0
- added joint joint1: type revolute, parent base, child link1, origin xyz=0 0 0.1575 rpy=0 0 0, axis 0 0 1, limit lower=-2.96706 upper=2.96706 effort=320 velocity=1.4835
- added joint joint2: type revolute, parent link1, child link2, origin xyz=0 0 0.2025 rpy=1.5708 0 3.14159, axis 0 0 1, limit lower=-2.0944 upper=2.0944 effort=320 velocity=1.4835
- added joint joint3: type revolute, parent link2, child link3, origin xyz=0 0.2045 0 rpy=1.5708 0 3.14159, axis 0 0 1, limit lower=-2.96706 upper=2.96706 effort=176 velocity=1.7453
- added joint joint4: type revolute, parent link3, child link4, origin xyz=0 0 0.2155 rpy=1.5708 0 0, axis 0 0 1, limit lower=-2.0944 upper=2.0944 effort=176 velocity=1.3090
- added joint joint5: type revolute, parent link4, child link5, origin xyz=0 0.1845 0 rpy=1.5708 0 3.14159, axis 0 0 1, limit lower=-2.96706 upper=2.96706 effort=110 velocity=2.2689
- added joint joint6: type revolute, parent link5, child link6, origin xyz=0 0 0.2155 rpy=1.5708 0 0, axis 0 0 1, limit lower=-2.0944 upper=2.0944 effort=40 velocity=2.3562
- added joint joint7: type revolute, parent link6, child link7, origin xyz=0 0.081 0 rpy=1.5708 0 3.14159, axis 0 0 1, limit lower=-3.05433 upper=3.05433 effort=40 velocity=2.3562
- joint iiwa_joint_ee: parent iiwa_link_7 -> link7

File: resources/iiwa/iiwa_spherized.urdf (robot description, URDF)
Before this commit: robot iiwa, 21 links, 20 joints
Links:
- removed link iiwa_link_0
- removed link iiwa_link_1
- removed link iiwa_link_2
- removed link iiwa_link_3
- removed link iiwa_link_4
- removed link iiwa_link_5
- removed link iiwa_link_6
- removed link iiwa_link_7
- removed link world
- added link attachment_site
- added link base, mass 5; collision sphere radius=0.07; visual mesh filename=assets/link_0.obj
- added link link1, mass 5.76; collision sphere radius=0.07; collision sphere radius=0.07
- added link link2, mass 6.35; collision sphere radius=0.065; collision sphere radius=0.065
- added link link3, mass 3.5; collision sphere radius=0.055; collision sphere radius=0.055
- added link link4, mass 3.5; collision sphere radius=0.06; collision sphere radius=0.06
- added link link5, mass 3.5; collision sphere radius=0.035; collision sphere radius=0.035
- added link link6, mass 1.8; collision sphere radius=0.055; collision sphere radius=0.065
- added link link7, mass 1.2; collision sphere radius=0.02; visual mesh filename=assets/link_7.obj
Joints:
- removed joint iiwa_joint_1
- removed joint iiwa_joint_2
- removed joint iiwa_joint_3
- removed joint iiwa_joint_4
- removed joint iiwa_joint_5
- removed joint iiwa_joint_6
- removed joint iiwa_joint_7
- removed joint world_iiwa_joint
- added joint attachment_joint: type fixed, parent link7, child attachment_site, origin xyz=0 0 0.045 rpy=0 0 0
- added joint joint1: type revolute, parent base, child link1, origin xyz=0 0 0.1575 rpy=0 0 0, axis 0 0 1, limit lower=-2.96706 upper=2.96706 effort=320 velocity=1.4835
- added joint joint2: type revolute, parent link1, child link2, origin xyz=0 0 0.2025 rpy=1.5708 0 3.14159, axis 0 0 1, limit lower=-2.0944 upper=2.0944 effort=320 velocity=1.4835
- added joint joint3: type revolute, parent link2, child link3, origin xyz=0 0.2045 0 rpy=1.5708 0 3.14159, axis 0 0 1, limit lower=-2.96706 upper=2.96706 effort=176 velocity=1.7453
- added joint joint4: type revolute, parent link3, child link4, origin xyz=0 0 0.2155 rpy=1.5708 0 0, axis 0 0 1, limit lower=-2.0944 upper=2.0944 effort=176 velocity=1.3090
- added joint joint5: type revolute, parent link4, child link5, origin xyz=0 0.1845 0 rpy=1.5708 0 3.14159, axis 0 0 1, limit lower=-2.96706 upper=2.96706 effort=110 velocity=2.2689
- added joint joint6: type revolute, parent link5, child link6, origin xyz=0 0 0.2155 rpy=1.5708 0 0, axis 0 0 1, limit lower=-2.0944 upper=2.0944 effort=40 velocity=2.3562
- added joint joint7: type revolute, parent link6, child link7, origin xyz=0 0.081 0 rpy=1.5708 0 3.14159, axis 0 0 1, limit lower=-3.05433 upper=3.05433 effort=40 velocity=2.3562
- joint iiwa_joint_ee: parent iiwa_link_7 -> link7

Commit message: remove bbase sphere

File: cricket/resources/iiwa/iiwa_spherized.urdf (robot description, URDF)
Before this commit: robot iiwa14, 21 links, 20 joints
Links:
- link base: geometry visual mesh filename=assets/link_0.obj

File: resources/iiwa/iiwa_spherized.urdf (robot description, URDF)
Before this commit: robot iiwa14, 21 links, 20 joints
Links:
- link base: geometry visual mesh filename=assets/link_0.obj
- link link1: geometry collision sphere radius=0.07; collision sphere radius=0.07
- link link2: geometry collision sphere radius=0.065; collision sphere radius=0.065
- link link3: geometry collision sphere radius=0.055; collision sphere radius=0.055
- link link4: geometry collision sphere radius=0.06; collision sphere radius=0.06
- link link5: geometry collision sphere radius=0.035; collision sphere radius=0.035
- link link6: geometry collision sphere radius=0.055; collision sphere radius=0.065
- link link7: geometry collision sphere radius=0.02; visual mesh filename=assets/link_7.obj
